Commit message: basic support for cartesian motion, additional frame to represent ur internal frames, additional action for commanding cartesiantrajectories

File: ur_description/urdf/ur5.urdf.xacro (robot description, xacro)
@@ -87,8 +87,14 @@
       </xacro:cylinder_inertial>
     </link>
+    <link name="${prefix}ur_base_link"/>
+    <joint name="${prefix}ur_base_joint" type="fixed">
+      <parent link="${prefix}base_link" />
+      <child link = "${prefix}ur_base_link" />
+      <origin xyz="0.0 0.0 0.0" rpy="0.0 0.0 -${pi}" />
+    </joint>
     <joint name="${prefix}shoulder_pan_joint" type="revolute">
-      <parent link="${prefix}base_link" />
+      <parent link="${prefix}ur_base_link" />
       <child link = "${prefix}shoulder_link" />
-      <origin xyz="0.0 0.0 ${shoulder_height}" rpy="0.0 0.0 0.0" />
+      <origin xyz="0.0 0.0 ${shoulder_height}" rpy="0.0 0.0 ${pi}" />
       <axis xyz="0 0 1" />
       <xacro:unless value="${joint_limited}">
@@ -273,8 +279,14 @@
       </xacro:cylinder_inertial>
     </link>
+    <joint name="${prefix}ur_ee_joint" type="fixed">
+      <parent link="${prefix}wrist_3_link" />
+      <child link = "${prefix}ur_ee_link" />
+      <origin xyz="0.0 ${wrist_3_length} 0.0" rpy="-${pi/2.0} 0.0 0.0" />
+    </joint>
+    <link name="${prefix}ur_ee_link"/>
     <joint name="${prefix}ee_fixed_joint" type="fixed">
-      <parent link="${prefix}wrist_3_link" />
+      <parent link="${prefix}ur_ee_link" />
       <child link = "${prefix}ee_link" />
-      <origin xyz="0.0 ${wrist_3_length} 0.0" rpy="0.0 0.0 ${pi/2.0}" />
+      <origin xyz="0.0 0.0 0.0" rpy="${pi/2.0} -${pi/2.0} 0.0" />
     </joint>
     <link name="${prefix}ee_link">

Commit message: adding artificial link for moveit collision detection

File: ur_description/urdf/ur5.urdf.xacro (robot description, xacro)
@@ -284,5 +284,12 @@
       <origin xyz="0.0 ${wrist_3_length} 0.0" rpy="-${pi/2.0} 0.0 0.0" />
     </joint>
-    <link name="${prefix}ur_ee_link"/>
+    <link name="${prefix}ur_ee_link">
+	  <collision>
+        <geometry>
+          <box size="0.01 0.01 0.01"/>
+        </geometry>
+        <origin rpy="0 0 0" xyz="0 0 -0.01"/>
+      </collision>
+    </link>
     <joint name="${prefix}ee_fixed_joint" type="fixed">
       <parent link="${prefix}ur_ee_link" />
